Commit message: gazeboカクカクなのを調査

File: models/omni_robot/lidar.xacro (robot description, xacro)
@@ -1,5 +1,5 @@
 <?xml version="1.0"?>
 <robot xmlns:xacro="http://ros.org/wiki/xacro">
-  <xacro:macro name="lidar_macro" params="parent prefix xyz rpy angle_min angle_max">
+  <xacro:macro name="lidar_macro" params="parent prefix xyz rpy angle_min angle_max visualize update_rate samples">
     <joint name="${prefix}_joint" type="fixed">
       <parent link="${parent}"/>
@@ -31,6 +31,6 @@
         <pose>0 0 0.025 0 0 0</pose>
         <always_on>true</always_on>
-        <visualize>true</visualize>
-        <update_rate>20</update_rate>
+        <visualize>${visualize}</visualize>
+        <update_rate>${update_rate}</update_rate>
         <topic>/scan</topic>
         <gz_frame_id>${prefix}_link</gz_frame_id>
@@ -38,5 +38,5 @@
           <scan>
             <horizontal>
-              <samples>1440</samples>
+              <samples>${samples}</samples>
               <resolution>1</resolution>
               <min_angle>${angle_min}</min_angle>

File: models/omni_robot/urdf/omni_robot.xacro (robot description, xacro)
@@ -1,4 +1,8 @@
 <?xml version="1.0"?>
 <robot xmlns:xacro="http://www.ros.org/wiki/xacro" name="omni_robot">
+  <xacro:arg name="enable_lidar" default="true"/>
+  <xacro:arg name="lidar_visualize" default="true"/>
+  <xacro:arg name="lidar_update_rate" default="20"/>
+  <xacro:arg name="lidar_samples" default="1440"/>
   <xacro:include filename="$(find gazebo_simulator)/models/omni_robot/omni_common.xacro"/>
   <xacro:include filename="$(find gazebo_simulator)/models/omni_robot/omni_wheel.xacro"/>
@@ -34,11 +38,16 @@
     </inertial>
   </link>
-  <xacro:lidar_macro
-    prefix="lidar"
-    parent="base_link"
-    xyz="-0.3 0 -0.075"
-    rpy="0 0 0"
-    angle_min="${80 * pi / 180}"
-    angle_max="${280 * pi / 180}"/>
+  <xacro:if value="$(arg enable_lidar)">
+    <xacro:lidar_macro
+      prefix="lidar"
+      parent="base_link"
+      xyz="-0.3 0 -0.075"
+      rpy="0 0 0"
+      angle_min="${80 * pi / 180}"
+      angle_max="${280 * pi / 180}"
+      visualize="$(arg lidar_visualize)"
+      update_rate="$(arg lidar_update_rate)"
+      samples="$(arg lidar_samples)"/>
+  </xacro:if>
   <joint name="wheel0_attach_joint" type="fixed">
     <parent link="base_link"/>
