Commit message: mecanumモデルを修正

File: models/mecanum/urdf/materials.xacro (robot description, xacro)
@@ -1,4 +1,4 @@
 <?xml version="1.0" ?>
-<robot name="wheel_final" xmlns:xacro="http://www.ros.org/wiki/xacro" >
+<robot name="mecanum" xmlns:xacro="http://www.ros.org/wiki/xacro" >
 <material name="silver_default">
   <color rgba="0.700 0.700 0.700 1.000"/>

File: models/mecanum/urdf/mecanum.xacro (robot description, xacro)
@@ -1,4 +1,4 @@
 <?xml version="1.0" ?>
-<robot name="wheel_final" xmlns:xacro="http://www.ros.org/wiki/xacro">
+<robot name="mecanum" xmlns:xacro="http://www.ros.org/wiki/xacro">
 <xacro:property name="robot_name" value="$(arg robot_name)"/>
 <xacro:include filename="$(find gazebo_simulator)/models/${robot_name}/urdf/materials.xacro" />
@@ -13,5 +13,5 @@
     <origin xyz="0 0 0" rpy="0 0 0"/>
     <geometry>
-      <mesh filename="package://wheel_final/meshes/base_link.stl" scale="0.001 0.001 0.001"/>
+      <mesh filename="package://mecanum/meshes/base_link.stl" scale="0.001 0.001 0.001"/>
     </geometry>
     <material name="opaque202209238"/>
@@ -20,5 +20,5 @@
     <origin xyz="0 0 0" rpy="0 0 0"/>
     <geometry>
-      <mesh filename="package://wheel_final/meshes/base_link.stl" scale="0.001 0.001 0.001"/>
+      <mesh filename="package://mecanum/meshes/base_link.stl" scale="0.001 0.001 0.001"/>
     </geometry>
   </collision>
