Commit message: メカなむモデルを更新

File: models/mecanum_module/urdf/materials.xacro (robot description, xacro)
@@ -4,4 +4,13 @@
   <color rgba="0.700 0.700 0.700 1.000"/>
 </material>
+<material name="opaque202209238">
+  <color rgba="0.792156862745098 0.8196078431372549 0.9333333333333333 1.0"/>
+</material>
+<material name="opaque767676">
+  <color rgba="0.2980392156862745 0.2980392156862745 0.2980392156862745 1.0"/>
+</material>
+<material name="opaque255255255">
+  <color rgba="1.0 1.0 1.0 1.0"/>
+</material>
 <material name="_">
   <color rgba="0.6274509803921569 0.6274509803921569 0.6274509803921569 1.0"/>

File: models/mecanum_module/urdf/mecanum_module.xacro (robot description, xacro)
@@ -6,7 +6,7 @@
 <link name="base_link">
   <inertial>
-    <origin xyz="0.015 0.015 0.030616438356164385" rpy="0 0 0"/>
+    <origin xyz="0.013930521220351077 0.015409571278913166 0.05867537985716325" rpy="0 0 0"/>
     <mass value="0.4297875"/>
-    <inertia ixx="0.000171" iyy="0.000171" izz="6.4e-05" ixy="0.0" iyz="0.0" ixz="0.0"/>
+    <inertia ixx="0.000171" iyy="0.000171" izz="6.4e-05" ixy="-0.0" iyz="-0.0" ixz="0.0"/>
   </inertial>
   <visual>
