Commit message: メカナムのモデルを更新

File: models/mecanum_module/urdf/mecanum_module.xacro (robot description, xacro)
@@ -1,4 +1,4 @@
 <?xml version="1.0" ?>
-<robot name="mecanum" xmlns:xacro="http://www.ros.org/wiki/xacro">
+<robot name="mecanum_module" xmlns:xacro="http://www.ros.org/wiki/xacro">
 <xacro:property name="robot_name" value="$(arg robot_name)"/>
 <xacro:include filename="$(find gazebo_simulator)/models/${robot_name}/urdf/materials.xacro" />
@@ -6,19 +6,19 @@
 <link name="base_link">
   <inertial>
-    <origin xyz="0.03893052122041182 0.04540957127891325 0.11673602628480363" rpy="0 0 0"/>
-    <mass value="0.15456797657506838"/>
-    <inertia ixx="0.000139" iyy="0.000139" izz="0.000278" ixy="0.0" iyz="-0.0" ixz="-0.0"/>
+    <origin xyz="0.015 0.015 0.030616438356164385" rpy="0 0 0"/>
+    <mass value="0.4297875"/>
+    <inertia ixx="0.000171" iyy="0.000171" izz="6.4e-05" ixy="0.0" iyz="0.0" ixz="0.0"/>
   </inertial>
   <visual>
     <origin xyz="0 0 0" rpy="0 0 0"/>
     <geometry>
-      <mesh filename="package://mecanum/meshes/base_link.stl" scale="0.001 0.001 0.001"/>
+      <mesh filename="package://mecanum_module/meshes/base_link.stl" scale="0.001 0.001 0.001"/>
     </geometry>
-    <material name="opaque202209238"/>
+    <material name="_"/>
   </visual>
   <collision>
     <origin xyz="0 0 0" rpy="0 0 0"/>
     <geometry>
-      <mesh filename="package://mecanum/meshes/base_link.stl" scale="0.001 0.001 0.001"/>
+      <mesh filename="package://mecanum_module/meshes/base_link.stl" scale="0.001 0.001 0.001"/>
     </geometry>
   </collision>

Commit message: 4輪メカなむモデルを追加

File: models/mecanum_module/urdf/mecanum_module.xacro (robot description, xacro)
@@ -6,359 +6,1473 @@
 <link name="base_link">
   <inertial>
-    <origin xyz="0.015 0.015 0.030616438356164385" rpy="0 0 0"/>
+    <origin xyz="0.25 0.25 0.0025" rpy="0 0 0"/>
+    <mass value="9.8125"/>
+    <inertia ixx="0.204448" iyy="0.204448" izz="0.408854" ixy="0.0" iyz="0.0" ixz="0.0"/>
+  </inertial>
+  <visual>
+    <origin xyz="0 0 0" rpy="0 0 0"/>
+    <geometry>
+      <mesh filename="package://mecanum_module/meshes/base_link.stl" scale="0.001 0.001 0.001"/>
+    </geometry>
+    <material name="_"/>
+  </visual>
+  <collision>
+    <origin xyz="0 0 0" rpy="0 0 0"/>
+    <geometry>
+      <mesh filename="package://mecanum_module/meshes/base_link.stl" scale="0.001 0.001 0.001"/>
+    </geometry>
+  </collision>
+</link>
+<link name="mecanum_module_plate_1">
+  <inertial>
+    <origin xyz="-0.0006770847837933719 -8.222589276130066e-15 5.2496201830010136e-14" rpy="0 0 0"/>
+    <mass value="0.1545679765750766"/>
+    <inertia ixx="0.000278" iyy="0.000139" izz="0.000139" ixy="-0.0" iyz="-0.0" ixz="0.0"/>
+  </inertial>
+  <visual>
+    <origin xyz="0.05 -0.04 -0.02" rpy="0 0 0"/>
+    <geometry>
+      <mesh filename="package://mecanum_module/meshes/mecanum_module_plate_1.stl" scale="0.001 0.001 0.001"/>
+    </geometry>
+    <material name="opaque202209238"/>
+  </visual>
+  <collision>
+    <origin xyz="0.05 -0.04 -0.02" rpy="0 0 0"/>
+    <geometry>
+      <mesh filename="package://mecanum_module/meshes/mecanum_module_plate_1.stl" scale="0.001 0.001 0.001"/>
+    </geometry>
+  </collision>
+</link>
+<link name="mecanum_module_roller_1">
+  <inertial>
+    <origin xyz="0.018314100662847114 0.007470946457023422 0.016721067976369994" rpy="0 0 0"/>
+    <mass value="0.09313994123705087"/>
+    <inertia ixx="1.1e-05" iyy="1.7e-05" izz="1.2e-05" ixy="-3e-06" iyz="-3e-06" ixz="-7e-06"/>
+  </inertial>
+  <visual>
+    <origin xyz="0.043883 0.017417 -0.025578" rpy="0 0 0"/>
+    <geometry>
+      <mesh filename="package://mecanum_module/meshes/mecanum_module_roller_1.stl" scale="0.001 0.001 0.001"/>
+    </geometry>
+    <material name="opaque767676"/>
+  </visual>
+  <collision>
+    <origin xyz="0.043883 0.017417 -0.025578" rpy="0 0 0"/>
+    <geometry>
+      <mesh filename="package://mecanum_module/meshes/mecanum_module_roller_1.stl" scale="0.001 0.001 0.001"/>
+    </geometry>
+  </collision>
+</link>
+<link name="mecanum_module_roller_2">
+  <inertial>
+    <origin xyz="0.01838481134096658 -0.00189838570793922 0.01828686537296428" rpy="0 0 0"/>
+    <mass value="0.09313994123705087"/>
+    <inertia ixx="1.1e-05" iyy="1.8e-05" izz="1.1e-05" ixy="1e-06" iyz="1e-06" ixz="-7e-06"/>
+  </inertial>
+  <visual>
+    <origin xyz="0.043883 0.012513 0.003878" rpy="0 0 0"/>
+    <geometry>
+      <mesh filename="package://mecanum_module/meshes/mecanum_module_roller_2.stl" scale="0.001 0.001 0.001"/>
+    </geometry>
+    <material name="opaque767676"/>
+  </visual>
+  <collision>
+    <origin xyz="0.043883 0.012513 0.003878" rpy="0 0 0"/>
+    <geometry>
+      <mesh filename="package://mecanum_module/meshes/mecanum_module_roller_2.stl" scale="0.001 0.001 0.001"/>
+    </geometry>
+  </collision>
+</link>
+<link name="mecanum_module_roller_3">
+  <inertial>
+    <origin xyz="0.018384811340966856 -0.010787074964667957 0.014887242523040436" rpy="0 0 0"/>
+    <mass value="0.09313994123705087"/>
+    <inertia ixx="1.1e-05" iyy="1.6e-05" izz="1.4e-05" ixy="4e-06" iyz="3e-06" ixz="-6e-06"/>
+  </inertial>
+  <visual>
+    <origin xyz="0.043883 -0.006461 0.026935" rpy="0 0 0"/>
+    <geometry>
+      <mesh filename="package://mecanum_module/meshes/mecanum_module_roller_3.stl" scale="0.001 0.001 0.001"/>
+    </geometry>
+    <material name="opaque767676"/>
+  </visual>
+  <collision>
+    <origin xyz="0.043883 -0.006461 0.026935" rpy="0 0 0"/>
+    <geometry>
+      <mesh filename="package://mecanum_module/meshes/mecanum_module_roller_3.stl" scale="0.001 0.001 0.001"/>
+    </geometry>
+  </collision>
+</link>
+<link name="mecanum_module_roller_4">
+  <inertial>
+    <origin xyz="0.01838481134096841 -0.016785628230974146 0.007499790408296861" rpy="0 0 0"/>
+    <mass value="0.09313994123705087"/>
+    <inertia ixx="1.1e-05" iyy="1.2e-05" izz="1.7e-05" ixy="7e-06" iyz="3e-06" ixz="-3e-06"/>
+  </inertial>
+  <visual>
+    <origin xyz="0.043883 -0.034422 0.037417" rpy="0 0 0"/>
+    <geometry>
+      <mesh filename="package://mecanum_module/meshes/mecanum_module_roller_4.stl" scale="0.001 0.001 0.001"/>
+    </geometry>
+    <material name="opaque767676"/>
+  </visual>
+  <collision>
+    <origin xyz="0.043883 -0.034422 0.037417" rpy="0 0 0"/>
+    <geometry>
+      <mesh filename="package://mecanum_module/meshes/mecanum_module_roller_4.stl" scale="0.001 0.001 0.001"/>
+    </geometry>
+  </collision>
+</link>
+<link name="mecanum_module_roller_5">
+  <inertial>
+    <origin xyz="0.018384811340970468 -0.018286865372961286 -0.0018983857079341374" rpy="0 0 0"/>
+    <mass value="0.09313994123705087"/>
+    <inertia ixx="1.1e-05" iyy="1.1e-05" izz="1.8e-05" ixy="7e-06" iyz="-1e-06" ixz="1e-06"/>
+  </inertial>
+  <visual>
+    <origin xyz="0.043883 -0.063878 0.032513" rpy="0 0 0"/>
+    <geometry>
+      <mesh filename="package://mecanum_module/meshes/mecanum_module_roller_5.stl" scale="0.001 0.001 0.001"/>
+    </geometry>
+    <material name="opaque767676"/>
+  </visual>
+  <collision>
+    <origin xyz="0.043883 -0.063878 0.032513" rpy="0 0 0"/>
+    <geometry>
+      <mesh filename="package://mecanum_module/meshes/mecanum_module_roller_5.stl" scale="0.001 0.001 0.001"/>
+    </geometry>
+  </collision>
+</link>
+<link name="mecanum_module_roller_6">
+  <inertial>
+    <origin xyz="0.018384811340971613 -0.01488724252303647 -0.010787074964665177" rpy="0 0 0"/>
+    <mass value="0.09313994123705087"/>
+    <inertia ixx="1.1e-05" iyy="1.4e-05" izz="1.6e-05" ixy="6e-06" iyz="-3e-06" ixz="4e-06"/>
+  </inertial>
+  <visual>
+    <origin xyz="0.043883 -0.086935 0.013539" rpy="0 0 0"/>
+    <geometry>
+      <mesh filename="package://mecanum_module/meshes/mecanum_module_roller_6.stl" scale="0.001 0.001 0.001"/>
+    </geometry>
+    <material name="opaque767676"/>
+  </visual>
+  <collision>
+    <origin xyz="0.043883 -0.086935 0.013539" rpy="0 0 0"/>
+    <geometry>
+      <mesh filename="package://mecanum_module/meshes/mecanum_module_roller_6.stl" scale="0.001 0.001 0.001"/>
+    </geometry>
+  </collision>
+</link>
+<link name="mecanum_module_roller_7">
+  <inertial>
+    <origin xyz="0.0183848113409725 -0.007499790408291879 -0.01678562823097173" rpy="0 0 0"/>
+    <mass value="0.09313994123705087"/>
+    <inertia ixx="1.1e-05" iyy="1.7e-05" izz="1.2e-05" ixy="3e-06" iyz="-3e-06" ixz="7e-06"/>
+  </inertial>
+  <visual>
+    <origin xyz="0.043883 -0.097417 -0.014422" rpy="0 0 0"/>
+    <geometry>
+      <mesh filename="package://mecanum_module/meshes/mecanum_module_roller_7.stl" scale="0.001 0.001 0.001"/>
+    </geometry>
+    <material name="opaque767676"/>
+  </visual>
+  <collision>
+    <origin xyz="0.043883 -0.097417 -0.014422" rpy="0 0 0"/>
+    <geometry>
+      <mesh filename="package://mecanum_module/meshes/mecanum_module_roller_7.stl" scale="0.001 0.001 0.001"/>
+    </geometry>
+  </collision>
+</link>
+<link name="mecanum_module_roller_8">
+  <inertial>
+    <origin xyz="0.01838481134097244 0.0018983857079400007 -0.018286865372958056" rpy="0 0 0"/>
+    <mass value="0.09313994123705087"/>
+    <inertia ixx="1.1e-05" iyy="1.8e-05" izz="1.1e-05" ixy="-1e-06" iyz="1e-06" ixz="7e-06"/>
+  </inertial>
+  <visual>
+    <origin xyz="0.043883 -0.092513 -0.043878" rpy="0 0 0"/>
+    <geometry>
+      <mesh filename="package://mecanum_module/meshes/mecanum_module_roller_8.stl" scale="0.001 0.001 0.001"/>
+    </geometry>
+    <material name="opaque767676"/>
+  </visual>
+  <collision>
+    <origin xyz="0.043883 -0.092513 -0.043878" rpy="0 0 0"/>
+    <geometry>
+      <mesh filename="package://mecanum_module/meshes/mecanum_module_roller_8.stl" scale="0.001 0.001 0.001"/>
+    </geometry>
+  </collision>
+</link>
+<link name="mecanum_module_roller_9">
+  <inertial>
+    <origin xyz="0.018384811340971377 0.010787074964671003 -0.014887242523032418" rpy="0 0 0"/>
+    <mass value="0.09313994123705087"/>
+    <inertia ixx="1.1e-05" iyy="1.6e-05" izz="1.4e-05" ixy="-4e-06" iyz="3e-06" ixz="6e-06"/>
+  </inertial>
+  <visual>
+    <origin xyz="0.043883 -0.073539 -0.066935" rpy="0 0 0"/>
+    <geometry>
+      <mesh filename="package://mecanum_module/meshes/mecanum_module_roller_9.stl" scale="0.001 0.001 0.001"/>
+    </geometry>
+    <material name="opaque767676"/>
+  </visual>
+  <collision>
+    <origin xyz="0.043883 -0.073539 -0.066935" rpy="0 0 0"/>
+    <geometry>
+      <mesh filename="package://mecanum_module/meshes/mecanum_module_roller_9.stl" scale="0.001 0.001 0.001"/>
+    </geometry>
+  </collision>
+</link>
+<link name="mecanum_module_roller_10">
+  <inertial>
+    <origin xyz="0.018384811340969892 0.016785628230976644 -0.00749979040828741" rpy="0 0 0"/>
+    <mass value="0.09313994123705087"/>
+    <inertia ixx="1.1e-05" iyy="1.2e-05" izz="1.7e-05" ixy="-7e-06" iyz="3e-06" ixz="3e-06"/>
+  </inertial>
+  <visual>
+    <origin xyz="0.043883 -0.045578 -0.077417" rpy="0 0 0"/>
+    <geometry>
+      <mesh filename="package://mecanum_module/meshes/mecanum_module_roller_10.stl" scale="0.001 0.001 0.001"/>
+    </geometry>
+    <material name="opaque767676"/>
+  </visual>
+  <collision>
+    <origin xyz="0.043883 -0.045578 -0.077417" rpy="0 0 0"/>
+    <geometry>
+      <mesh filename="package://mecanum_module/meshes/mecanum_module_roller_10.stl" scale="0.001 0.001 0.001"/>
+    </geometry>
+  </collision>
+</link>
+<link name="mecanum_module_roller_11">
+  <inertial>
+    <origin xyz="0.018384811340968178 0.018286865372962067 0.0018983857079439004" rpy="0 0 0"/>
+    <mass value="0.09313994123705087"/>
+    <inertia ixx="1.1e-05" iyy="1.1e-05" izz="1.8e-05" ixy="-7e-06" iyz="-1e-06" ixz="-1e-06"/>
+  </inertial>
+  <visual>
+    <origin xyz="0.043883 -0.016122 -0.072513" rpy="0 0 0"/>
+    <geometry>
+      <mesh filename="package://mecanum_module/meshes/mecanum_module_roller_11.stl" scale="0.001 0.001 0.001"/>
+    </geometry>
+    <material name="opaque767676"/>
+  </visual>
+  <collision>
+    <origin xyz="0.043883 -0.016122 -0.072513" rpy="0 0 0"/>
+    <geometry>
+      <mesh filename="package://mecanum_module/meshes/mecanum_module_roller_11.stl" scale="0.001 0.001 0.001"/>
+    </geometry>
+  </collision>
+</link>
+<link name="mecanum_module_roller_12">
+  <inertial>
+    <origin xyz="0.018314100662847988 0.014829982801187448 0.010745586119742065" rpy="0 0 0"/>
+    <mass value="0.09313994123705087"/>
+    <inertia ixx="1.1e-05" iyy="1.4e-05" izz="1.6e-05" ixy="-6e-06" iyz="-3e-06" ixz="-4e-06"/>
+  </inertial>
+  <visual>
+    <origin xyz="0.043883 0.006935 -0.053539" rpy="0 0 0"/>
+    <geometry>
+      <mesh filename="package://mecanum_module/meshes/mecanum_module_roller_12.stl" scale="0.001 0.001 0.001"/>
+    </geometry>
+    <material name="opaque767676"/>
+  </visual>
+  <collision>
+    <origin xyz="0.043883 0.006935 -0.053539" rpy="0 0 0"/>
+    <geometry>
+      <mesh filename="package://mecanum_module/meshes/mecanum_module_roller_12.stl" scale="0.001 0.001 0.001"/>
+    </geometry>
+  </collision>
+</link>
+<link name="mecanum_module_plate_r_1">
+  <inertial>
+    <origin xyz="-0.0006770847838043145 0.0 -1.214306433183765e-16" rpy="0 0 0"/>
+    <mass value="0.30913595315013653"/>
+    <inertia ixx="0.000556" iyy="0.000279" izz="0.000279" ixy="0.0" iyz="-0.0" ixz="0.0"/>
+  </inertial>
+  <visual>
+    <origin xyz="0.05 -0.46 -0.02" rpy="0 0 0"/>
+    <geometry>
+      <mesh filename="package://mecanum_module/meshes/mecanum_module_plate_r_1.stl" scale="0.001 0.001 0.001"/>
+    </geometry>
+    <material name="opaque202209238"/>
+  </visual>
+  <collision>
+    <origin xyz="0.05 -0.46 -0.02" rpy="0 0 0"/>
+    <geometry>
+      <mesh filename="package://mecanum_module/meshes/mecanum_module_plate_r_1.stl" scale="0.001 0.001 0.001"/>
+    </geometry>
+  </collision>
+</link>
+<link name="mecanum_module_roller_13">
+  <inertial>
+    <origin xyz="0.01838481134096692 -0.016785628230978122 -0.007499790408292573" rpy="0 0 0"/>
+    <mass value="0.09313994123705087"/>
+    <inertia ixx="1.1e-05" iyy="1.2e-05" izz="1.7e-05" ixy="7e-06" iyz="-3e-06" ixz="3e-06"/>
+  </inertial>
+  <visual>
+    <origin xyz="0.043883 -0.454422 -0.077417" rpy="0 0 0"/>
+    <geometry>
+      <mesh filename="package://mecanum_module/meshes/mecanum_module_roller_13.stl" scale="0.001 0.001 0.001"/>
+    </geometry>
+    <material name="opaque767676"/>
+  </visual>
+  <collision>
+    <origin xyz="0.043883 -0.454422 -0.077417" rpy="0 0 0"/>
+    <geometry>
+      <mesh filename="package://mecanum_module/meshes/mecanum_module_roller_13.stl" scale="0.001 0.001 0.001"/>
+    </geometry>
+  </collision>
+</link>
+<link name="mecanum_module_roller_14">
+  <inertial>
+    <origin xyz="0.01838481134096749 -0.010787074964672738 -0.014887242523036595" rpy="0 0 0"/>
+    <mass value="0.09313994123705087"/>
+    <inertia ixx="1.1e-05" iyy="1.6e-05" izz="1.4e-05" ixy="4e-06" iyz="-3e-06" ixz="6e-06"/>
+  </inertial>
+  <visual>
+    <origin xyz="0.043883 -0.426461 -0.066935" rpy="0 0 0"/>
+    <geometry>
+      <mesh filename="package://mecanum_module/meshes/mecanum_module_roller_14.stl" scale="0.001 0.001 0.001"/>
+    </geometry>
+    <material name="opaque767676"/>
+  </visual>
+  <collision>
+    <origin xyz="0.043883 -0.426461 -0.066935" rpy="0 0 0"/>
+    <geometry>
+      <mesh filename="package://mecanum_module/meshes/mecanum_module_roller_14.stl" scale="0.001 0.001 0.001"/>
+    </geometry>
+  </collision>
+</link>
+<link name="mecanum_module_roller_15">
+  <inertial>
+    <origin xyz="0.018384811340968688 -0.0018983857079427069 -0.018286865372962084" rpy="0 0 0"/>
+    <mass value="0.09313994123705087"/>
+    <inertia ixx="1.1e-05" iyy="1.8e-05" izz="1.1e-05" ixy="1e-06" iyz="-1e-06" ixz="7e-06"/>
+  </inertial>
+  <visual>
+    <origin xyz="0.043883 -0.407487 -0.043878" rpy="0 0 0"/>
+    <geometry>
+      <mesh filename="package://mecanum_module/meshes/mecanum_module_roller_15.stl" scale="0.001 0.001 0.001"/>
+    </geometry>
+    <material name="opaque767676"/>
+  </visual>
+  <collision>
+    <origin xyz="0.043883 -0.407487 -0.043878" rpy="0 0 0"/>
+    <geometry>
+      <mesh filename="package://mecanum_module/meshes/mecanum_module_roller_15.stl" scale="0.001 0.001 0.001"/>
+    </geometry>
+  </collision>
+</link>
+<link name="mecanum_module_roller_16">
+  <inertial>
+    <origin xyz="0.0183848113409701 0.007499790408288409 -0.016785628230976356" rpy="0 0 0"/>
+    <mass value="0.09313994123705087"/>
+    <inertia ixx="1.1e-05" iyy="1.7e-05" izz="1.2e-05" ixy="-3e-06" iyz="3e-06" ixz="7e-06"/>
+  </inertial>
+  <visual>
+    <origin xyz="0.043883 -0.402583 -0.014422" rpy="0 0 0"/>
+    <geometry>
+      <mesh filename="package://mecanum_module/meshes/mecanum_module_roller_16.stl" scale="0.001 0.001 0.001"/>
+    </geometry>
+    <material name="opaque767676"/>
+  </visual>
+  <collision>
+    <origin xyz="0.043883 -0.402583 -0.014422" rpy="0 0 0"/>
+    <geometry>
+      <mesh filename="package://mecanum_module/meshes/mecanum_module_roller_16.stl" scale="0.001 0.001 0.001"/>
+    </geometry>
+  </collision>
+</link>
+<link name="mecanum_module_roller_17">
+  <inertial>
+    <origin xyz="0.018384811340971235 0.014887242523033306 -0.010787074964670696" rpy="0 0 0"/>
+    <mass value="0.09313994123705087"/>
+    <inertia ixx="1.1e-05" iyy="1.4e-05" izz="1.6e-05" ixy="-6e-06" iyz="3e-06" ixz="4e-06"/>
+  </inertial>
+  <visual>
+    <origin xyz="0.043883 -0.413065 0.013539" rpy="0 0 0"/>
+    <geometry>
+      <mesh filename="package://mecanum_module/meshes/mecanum_module_roller_17.stl" scale="0.001 0.001 0.001"/>
+    </geometry>
+    <material name="opaque767676"/>
+  </visual>
+  <collision>
+    <origin xyz="0.043883 -0.413065 0.013539" rpy="0 0 0"/>
+    <geometry>
+      <mesh filename="package://mecanum_module/meshes/mecanum_module_roller_17.stl" scale="0.001 0.001 0.001"/>
+    </geometry>
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
Commit message: ジョイントの名前とモデルの名前が衝突している問題を修正

File: models/mecanum_module/urdf/mecanum_module.xacro (robot description, xacro)
@@ -604,5 +604,5 @@
   </collision>
 </link>
-<link name="motor_1">
+<link name="motor_body_1">
   <inertial>
     <origin xyz="-0.0006164383561644039 3.469446951953614e-17 0.014999999999999993" rpy="0 0 0"/>
@@ -613,5 +613,5 @@
     <origin xyz="-0.03 -0.04 -0.005" rpy="0 0 0"/>
     <geometry>
-      <mesh filename="package://mecanum_module/meshes/motor_1.stl" scale="0.001 0.001 0.001"/>
+      <mesh filename="package://mecanum_module/meshes/motor_body_1.stl" scale="0.001 0.001 0.001"/>
     </geometry>
     <material name="_"/>
@@ -620,9 +620,9 @@
     <origin xyz="-0.03 -0.04 -0.005" rpy="0 0 0"/>
     <geometry>
-      <mesh filename="package://mecanum_module/meshes/motor_1.stl" scale="0.001 0.001 0.001"/>
-    </geometry>
-  </collision>
-</link>
-<link name="motor_2">
+      <mesh filename="package://mecanum_module/meshes/motor_body_1.stl" scale="0.001 0.001 0.001"/>
+    </geometry>
+  </collision>
+</link>
+<link name="motor_body_2">
   <inertial>
     <origin xyz="-0.0006164383561643103 0.0 0.014999999999999947" rpy="0 0 0"/>
@@ -633,5 +633,5 @@
     <origin xyz="-0.03 -0.46 -0.005" rpy="0 0 0"/>
     <geometry>
-      <mesh filename="package://mecanum_module/meshes/motor_2.stl" scale="0.001 0.001 0.001"/>
+      <mesh filename="package://mecanum_module/meshes/motor_body_2.stl" scale="0.001 0.001 0.001"/>
     </geometry>
     <material name="_"/>
@@ -640,9 +640,9 @@
     <origin xyz="-0.03 -0.46 -0.005" rpy="0 0 0"/>
     <geometry>
-      <mesh filename="package://mecanum_module/meshes/motor_2.stl" scale="0.001 0.001 0.001"/>
-    </geometry>
-  </collision>
-</link>
-<link name="motor_3">
+      <mesh filename="package://mecanum_module/meshes/motor_body_2.stl" scale="0.001 0.001 0.001"/>
+    </geometry>
+  </collision>
+</link>
+<link name="motor_body_3">
   <inertial>
     <origin xyz="0.0006164383561643727 -1.1102230246251565e-16 0.014999999999999986" rpy="0 0 0"/>
@@ -653,5 +653,5 @@
     <origin xyz="-0.47 -0.46 -0.005" rpy="0 0 0"/>
     <geometry>
-      <mesh filename="package://mecanum_module/meshes/motor_3.stl" scale="0.001 0.001 0.001"/>
+      <mesh filename="package://mecanum_module/meshes/motor_body_3.stl" scale="0.001 0.001 0.001"/>
     </geometry>
     <material name="_"/>
@@ -660,9 +660,9 @@
     <origin xyz="-0.47 -0.46 -0.005" rpy="0 0 0"/>
     <geometry>
-      <mesh filename="package://mecanum_module/meshes/motor_3.stl" scale="0.001 0.001 0.001"/>
-    </geometry>
-  </collision>
-</link>
-<link name="motor_4">
+      <mesh filename="package://mecanum_module/meshes/motor_body_3.stl" scale="0.001 0.001 0.001"/>
+    </geometry>
+  </collision>
+</link>
+<link name="motor_body_4">
   <inertial>
     <origin xyz="0.0006164383561643727 2.7755575615628914e-17 0.014999999999999947" rpy="0 0 0"/>
@@ -673,5 +673,5 @@
     <origin xyz="-0.47 -0.04 -0.005" rpy="0 0 0"/>
     <geometry>
-      <mesh filename="package://mecanum_module/meshes/motor_4.stl" scale="0.001 0.001 0.001"/>
+      <mesh filename="package://mecanum_module/meshes/motor_body_4.stl" scale="0.001 0.001 0.001"/>
     </geometry>
     <material name="_"/>
@@ -680,5 +680,5 @@
     <origin xyz="-0.47 -0.04 -0.005" rpy="0 0 0"/>
     <geometry>
-      <mesh filename="package://mecanum_module/meshes/motor_4.stl" scale="0.001 0.001 0.001"/>
+      <mesh filename="package://mecanum_module/meshes/motor_body_4.stl" scale="0.001 0.001 0.001"/>
     </geometry>
   </collision>
@@ -1146,5 +1146,5 @@
 <joint name="motor_1" type="continuous">
   <origin xyz="-0.08 0.0 0.015" rpy="0 0 0"/>
-  <parent link="motor_1"/>
+  <parent link="motor_body_1"/>
   <child link="mecanum_module_plate_1"/>
   <axis xyz="-1.0 -0.0 0.0"/>
@@ -1224,5 +1224,5 @@
 <joint name="motor_2" type="continuous">
   <origin xyz="-0.08 0.0 0.015" rpy="0 0 0"/>
-  <parent link="motor_2"/>
+  <parent link="motor_body_2"/>
   <child link="mecanum_module_plate_r_1"/>
   <axis xyz="1.0 0.0 0.0"/>
@@ -1302,5 +1302,5 @@
 <joint name="motor_3" type="continuous">
   <origin xyz="0.08 0.0 0.015" rpy="0 0 0"/>
-  <parent link="motor_3"/>
+  <parent link="motor_body_3"/>
   <child link="mecanum_module_plate_2"/>
   <axis xyz="1.0 -0.0 0.0"/>
@@ -1314,5 +1314,5 @@
 <joint name="motor_4" type="continuous">
   <origin xyz="0.08 0.0 0.015" rpy="0 0 0"/>
-  <parent link="motor_4"/>
+  <parent link="motor_body_4"/>
   <child link="mecanum_module_plate_r_2"/>
   <axis xyz="-1.0 -0.0 0.0"/>
@@ -1321,20 +1321,20 @@
   <origin xyz="0.03 0.04 0.005" rpy="0 0 0"/>
   <parent link="base_link"/>
-  <child link="motor_1"/>
+  <child link="motor_body_1"/>
 </joint>
 <joint name="motor_lock_2" type="fixed">
   <origin xyz="0.03 0.46 0.005" rpy="0 0 0"/>
   <parent link="base_link"/>
-  <child link="motor_2"/>
+  <child link="motor_body_2"/>
 </joint>
 <joint name="motor_lock_3" type="fixed">
   <origin xyz="0.47 0.46 0.005" rpy="0 0 0"/>
   <parent link="base_link"/>
-  <child link="motor_3"/>
+  <child link="motor_body_3"/>
 </joint>
 <joint name="motor_lock_4" type="fixed">
   <origin xyz="0.47 0.04 0.005" rpy="0 0 0"/>
   <parent link="base_link"/>
-  <child link="motor_4"/>
+  <child link="motor_body_4"/>
 </joint>
 <joint name="roller3_2" type="continuous">
